File: ADC-Erweiterung/V0.1.sch (EAGLE design)
At the start: 16 parts, among them IC1 ADS124S0XIPBS, X1 32PIN-2.54, X2 MKDSN1,5/3-5,08

Commit message: :)
Parts:
- added C4: 100n, rcl:C-EUC0603
- added R10: 4.7k, rcl:R-EU_R0603
- added R11: 2k2, rcl:R-EU_R0805W
- added X3, X4, X5: A97581-ND, ADC-Erweiterung:A97581-ND
- C2: value 100n -> 330n
- X1: value 32PIN-2.54 -> 33PIN-2.54; device ADC-Erweiterung:32PIN-2.54 -> ADC-Erweiterung:33PIN-2.54
- X2: DIGIKEY_NR (none) -> 277-14503-ND; DIGIKEY_PRICE (none) -> 1.57
Connections:
- net GND: now also C1.2, C2.2, C4.2, R11.1, X3.2, X4.2, X5.2
- net N$10: now also R11.2
- net N$11: now also X5.1
- net N$12: now also X4.1
- net N$13: now also X3.1
- net N$8: now also R10.1
- net VCC: now also C1.1, C2.1, C4.1, R10.2
Other:
- moved on the sheet: C1, X2-1, X2-2, X2-3
