File: ADC-Erweiterung/V0.1.sch (EAGLE design)
At the start: 22 parts, among them IC1 ADS124S0XIPBS, X1 33PIN-2.54, X2 MKDSN1,5/3-5,08, X3 A97581-ND, X4 A97581-ND, X5 A97581-ND

Commit message: 2.5.19_BUP:)
Parts:
- removed R1: 47, rcl:R-EU_R0603
- added R12, R13, R14, R15, R16, R17: 4.7k, rcl:R-EU_R0603
- C1: value (none) -> 100n; DIGIKEY_NR (none) -> 1276-6439-1-ND; DIGIKEY_PRICE (none) -> 0.1
- C2: DIGIKEY_NR (none) -> 490-6050-1-ND; DIGIKEY_PRICE (none) -> .22
- C3: DIGIKEY_NR (none) -> 1276-1182-1-ND; DIGIKEY_PRIZE (none) -> 0.10 Fr.
- C4: DIGIKEY_NR (none) -> 1276-6439-1-ND; DIGIKEY_PRICE (none) -> 0.1
- R9: DIGIKEY_NR (none) -> 311-100DCT-ND; DIGIKEY_PRIZE (none) -> 0.20 Fr.
- X1: DIGIKEY_NR (none) -> 609-2223-ND; DIGIKEY_PRICE (none) -> 1.41 Fr.
Connections:
- new net N$16: IC1.AIN3, R15.2
- new net N$17: R16.1, X4.1
- new net N$18: R17.1, X3.1
- new net N$19: IC1.AIN2, R14.2
- new net N$20: IC1.AIN0, R12.2
- new net N$21: IC1.AIN1, R13.2
- net N$10: now also R14.1; no longer IC1.AIN2
- net N$11: now also R15.1; no longer IC1.AIN3
- net N$12: now also R16.2; no longer X4.1
- net N$13: now also R17.2; no longer X3.1
- net N$8: now also R12.1; no longer IC1.AIN0
- net N$9: now also R13.1; no longer IC1.AIN1
Other:
- note added: "stecker: Molec für pt100 paralell dazu"

Commit message: :-)
Parts:
- C3: DIGIKEY_PRICE (none) -> 0.10; DIGIKEY_PRIZE 0.10 Fr. -> (none)
- IC1: value ADS124S0XIPBS -> ADS124S06IPBS; DIGIKEY_NR (none) -> 296-45188-ND; DIGIKEY_PRICE (none) -> 10.15 Fr.
- LED1: DIGIKEY_NR (none) -> 475-3118-1-ND; DIGIKEY_PRICE (none) -> 0.52 Fr.
- R12: DIGIKEY_NR (none) -> 311-4.70KHRCT-ND; DIGIKEY_PRICE (none) -> 0.1
- R2: DIGIKEY_NR (none) -> 311-470GRCT-ND; DIGIKEY_PRICE (none) -> 0.1
- R9: DIGIKEY_PRICE (none) -> 0.20 Fr.; DIGIKEY_PRIZE 0.20 Fr. -> (none)
Other:
- moved on the sheet: C1, C2, C4, X1

Commit message: finished
Parts:
- added X6: MOLEX-8738-0343, ADC-Erweiterung:MOLEX-8738-0343
- C1, C4, R12, R2: DIGIKEY_PRICE 0.1 -> 0.10
- C2: DIGIKEY_PRICE .22 -> 0.22
- IC1: DIGIKEY_PRICE 10.15 Fr. -> 10.15
- LED1: DIGIKEY_PRICE 0.52 Fr. -> 0.52
- R10, R13, R14, R15, R16, R17: DIGIKEY_NR (none) -> 311-4.70KHRCT-ND; DIGIKEY_PRICE (none) -> 0.10
- R3, R4, R5, R6, R7, R8: DIGIKEY_NR (none) -> 311-470GRCT-ND; DIGIKEY_PRICE (none) -> 0.10
- R9: DIGIKEY_PRICE 0.20 Fr. -> 0.20
- X1: DIGIKEY_PRICE 1.41 Fr. -> 1.41
Connections:
- net N$10: now also X6.1
- net N$8: now also X6.3
- net N$9: now also X6.2

Commit message: :)
Other:
- note removed: "stecker: Molec für pt100 paralell dazu"
- moved on the sheet: C1, C2, C3, C4, IC1, LED1, R10, R11, R12, R13, R14, R15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

Commit message: Stand der Abgabe
Other:
- note added: "PT100"
- note removed: "TP100"
Changed lines of the file:
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@@
 <?xml version="1.0" encoding="utf-8"?>
 <!DOCTYPE eagle SYSTEM "eagle.dtd">
-<eagle version="9.3.0">
+<eagle version="9.2.1">
 <drawing>
 <settings>
@@
 <setting verticaltext="up"/>
 </settings>
-<grid distance="1.27" unitdist="mm" unit="mm" style="lines" multiple="1" display="no" altdistance="0.01" altunitdist="inch" altunit="inch"/>
+<grid distance="0.1" unitdist="inch" unit="inch" style="lines" multiple="1" display="no" altdistance="0.01" altunitdist="inch" altunit="inch"/>
 <layers>
 <layer number="1" name="Top" color="4" fill="1" visible="no" active="no"/>
@@
 <wire x1="19.05" y1="77.47" x2="19.05" y2="92.71" width="0.1524" layer="90"/>
 <wire x1="19.05" y1="92.71" x2="-3.81" y2="92.71" width="0.1524" layer="90"/>
-<text x="-3.81" y="92.71" size="1.6764" layer="90">TP100</text>
+<text x="-3.81" y="92.71" size="1.6764" layer="90">PT100</text>
 </plain>
 <instances>
@@
 <pinref part="X1" gate="G$1" pin="21"/>
 <wire x1="196.85" y1="48.26" x2="201.93" y2="48.26" width="0.1524" layer="91"/>
-<label x="201.93" y="48.26" size="0.6096" layer="95" xref="yes"/>
-</segment>
-<segment>
-<label x="143.51" y="67.31" size="0.6096" layer="95" xref="yes"/>
+<label x="201.93" y="48.26" size="0.8128" layer="95" xref="yes"/>
+</segment>
+<segment>
+<label x="143.51" y="67.31" size="0.8128" layer="95" xref="yes"/>
 <pinref part="R7" gate="G$1" pin="2"/>
 <wire x1="140.97" y1="67.31" x2="143.51" y2="67.31" width="0.1524" layer="91"/>
@@
 <net name="MOSI" class="0">
 <segment>
-<label x="143.51" y="72.39" size="0.6096" layer="95" xref="yes"/>
+<label x="143.51" y="72.39" size="0.8128" layer="95" xref="yes"/>
 <pinref part="R5" gate="G$1" pin="2"/>
 <wire x1="140.97" y1="72.39" x2="143.51" y2="72.39" width="0.1524" layer="91"/>
@@
 <pinref part="X1" gate="G$1" pin="22"/>
 <wire x1="196.85" y1="45.72" x2="201.93" y2="45.72" width="0.1524" layer="91"/>
-<label x="201.93" y="45.72" size="0.6096" layer="95" xref="yes"/>
+<label x="201.93" y="45.72" size="0.8128" layer="95" xref="yes"/>
 </segment>
 </net>
@@
 <pinref part="X1" gate="G$1" pin="23"/>
 <wire x1="196.85" y1="43.18" x2="201.93" y2="43.18" width="0.1524" layer="91"/>
-<label x="201.93" y="43.18" size="0.6096" layer="95" xref="yes"/>
-</segment>
-<segment>
-<label x="143.51" y="69.85" size="0.6096" layer="95" xref="yes"/>
+<label x="201.93" y="43.18" size="0.8128" layer="95" xref="yes"/>
+</segment>
+<segment>
+<label x="143.51" y="69.85" size="0.8128" layer="95" xref="yes"/>
 <pinref part="R6" gate="G$1" pin="2"/>
 <wire x1="140.97" y1="69.85" x2="143.51" y2="69.85" width="0.1524" layer="91"/>
@@
 <net name="START" class="0">
 <segment>
-<label x="143.51" y="80.01" size="0.6096" layer="95" xref="yes"/>
+<label x="143.51" y="80.01" size="0.8128" layer="95" xref="yes"/>
 <pinref part="R2" gate="G$1" pin="2"/>
 <wire x1="140.97" y1="80.01" x2="143.51" y2="80.01" width="0.1524" layer="91"/>
@@
 <pinref part="X1" gate="G$1" pin="25"/>
 <wire x1="196.85" y1="38.1" x2="201.93" y2="38.1" width="0.1524" layer="91"/>
-<label x="201.93" y="38.1" size="0.6096" layer="95" xref="yes"/>
+<label x="201.93" y="38.1" size="0.8128" layer="95" xref="yes"/>
 </segment>
 </net>
@@
 <pinref part="X1" gate="G$1" pin="24"/>
 <wire x1="196.85" y1="40.64" x2="201.93" y2="40.64" width="0.1524" layer="91"/>
-<label x="201.93" y="40.64" size="0.6096" layer="95" xref="yes"/>
-</segment>
-<segment>
-<label x="143.51" y="74.93" size="0.6096" layer="95" xref="yes"/>
+<label x="201.93" y="40.64" size="0.8128" layer="95" xref="yes"/>
+</segment>
+<segment>
+<label x="143.51" y="74.93" size="0.8128" layer="95" xref="yes"/>
 <pinref part="R4" gate="G$1" pin="2"/>
 <wire x1="140.97" y1="74.93" x2="143.51" y2="74.93" width="0.1524" layer="91"/>
@@
 <pinref part="X1" gate="G$1" pin="26"/>
 <wire x1="196.85" y1="35.56" x2="201.93" y2="35.56" width="0.1524" layer="91"/>
-<label x="201.93" y="35.56" size="0.6096" layer="95" xref="yes"/>
-</segment>
-<segment>
-<label x="143.51" y="77.47" size="0.6096" layer="95" xref="yes"/>
+<label x="201.93" y="35.56" size="0.8128" layer="95" xref="yes"/>
+</segment>
+<segment>
+<label x="143.51" y="77.47" size="0.8128" layer="95" xref="yes"/>
 <pinref part="R3" gate="G$1" pin="2"/>
 <wire x1="140.97" y1="77.47" x2="143.51" y2="77.47" width="0.1524" layer="91"/>
@@
 <pinref part="X1" gate="G$1" pin="27"/>
 <wire x1="196.85" y1="33.02" x2="201.93" y2="33.02" width="0.1524" layer="91"/>
-<label x="201.93" y="33.02" size="0.6096" layer="95" xref="yes"/>
-</segment>
-<segment>
-<label x="162.56" y="64.77" size="0.6096" layer="95" xref="yes"/>
+<label x="201.93" y="33.02" size="0.8128" layer="95" xref="yes"/>
+</segment>
+<segment>
+<label x="162.56" y="64.77" size="0.8128" layer="95" xref="yes"/>
 <pinref part="R8" gate="G$1" pin="2"/>
 <wire x1="158.75" y1="64.77" x2="162.56" y2="64.77" width="0.1524" layer="91"/>
