File: ADC-Erweiterung/V0.1.brd (EAGLE design)
At the start: 35.8 x 88.9 mm, 22 parts, among them IC1 ADS124S0XIPBS, X1 33PIN-2.54, X2 MKDSN1,5/3-5,08, X3 A97581-ND, X4 A97581-ND, X5 A97581-ND

Commit message: 2.5.19_BUP:)
Parts:
- removed R1: 47, rcl:R0603
- added R12, R13, R14, R15, R16, R17: 4.7k, rcl:R0603
- C1: value (none) -> 100n
- moved R6 0.76 mm to (22.6, 62.5)
Connections:
- new net N$16: IC1.4, R15.2
- new net N$17: R16.1, X4.1
- new net N$18: R17.1, X3.1
- new net N$19: IC1.5, R14.2
- new net N$20: IC1.7, R12.2
- new net N$21: IC1.6, R13.2
- net N$10: now also R14.1; no longer IC1.5
- net N$11: now also R15.1; no longer IC1.4
- net N$12: now also R16.2; no longer X4.1
- net N$13: now also R17.2; no longer X3.1
- net N$8: now also R12.1; no longer IC1.7
- net N$9: now also R13.1; no longer IC1.6
Routing:
- net N$13: track 73.8 -> 9.71 mm
- net N$18: track 0.00 -> 60.0 mm
- net N$12: track 67.8 -> 12.5 mm
- net N$17: track 0.00 -> 34.5 mm
- net N$16: track 0.00 -> 15.4 mm
- net N$11: track 28.1 -> 13.3 mm
- net N$10: track 20.4 -> 12.6 mm
- net N$8: track 28.0 -> 20.7 mm
- net N$19: track 0.00 -> 7.05 mm
- net N$9: track 18.7 -> 12.3 mm
- net N$20: track 0.00 -> 5.62 mm
- net N$21: track 0.00 -> 5.62 mm
- net N$6: track 8.88 -> 6.02 mm
- net N$5: track 4.77 -> 6.03 mm
- net MISO: track 37.7 -> 36.9 mm
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
Commit message: :-)
Parts:
- IC1: value ADS124S0XIPBS -> ADS124S06IPBS
Routing:
- net GND: track 30.2 -> 10.7 mm
- net N$18: track 60.0 -> 61.5 mm
Changed lines of the file:
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@@
 <grid distance="10" unitdist="mil" unit="mm" style="dots" multiple="1" display="yes" altdistance="5" altunitdist="mil" altunit="mil"/>
 <layers>
-<layer number="1" name="Top" color="4" fill="1" visible="no" active="yes"/>
+<layer number="1" name="Top" color="4" fill="1" visible="yes" active="yes"/>
 <layer number="2" name="Route2" color="16" fill="1" visible="no" active="no"/>
 <layer number="3" name="Route3" color="17" fill="1" visible="no" active="no"/>
@@
 <element name="C3" library="rcl" library_urn="urn:adsk.eagle:library:334" package="C0603" package3d_urn="urn:adsk.eagle:package:23616/2" value="1u" x="12.954" y="59.436" smashed="yes" rot="MR0">
 <attribute name="DIGIKEY_NR" value="1276-1182-1-ND" x="12.954" y="59.436" size="1.778" layer="28" rot="MR0" display="off"/>
-<attribute name="DIGIKEY_PRIZE" value="0.10 Fr." x="12.954" y="59.436" size="1.778" layer="28" rot="MR0" display="off"/>
+<attribute name="DIGIKEY_PRICE" value="0.10" x="12.954" y="59.436" size="1.778" layer="28" rot="MR0" display="off"/>
 <attribute name="NAME" x="13.589" y="61.595" size="1.27" layer="25" rot="R180"/>
 <attribute name="SPICEPREFIX" value="C" x="-25.146" y="13.716" size="1.778" layer="28" rot="MR0" display="off"/>
@@
 <attribute name="VALUE" x="13.843" y="83.439" size="1.27" layer="28" rot="MR90"/>
 </element>
-<element name="IC1" library="ADC-Erweiterung" package="TQFP32-05" value="ADS124S0XIPBS" x="14.732" y="65.024" smashed="yes" rot="MR270">
+<element name="IC1" library="ADC-Erweiterung" package="TQFP32-05" value="ADS124S06IPBS" x="14.732" y="65.024" smashed="yes" rot="MR270">
+<attribute name="DIGIKEY_NR" value="296-45188-ND" x="14.732" y="65.024" size="1.778" layer="28" rot="MR270" display="off"/>
+<attribute name="DIGIKEY_PRICE" value="10.15 Fr." x="14.732" y="65.024" size="1.778" layer="28" rot="MR270" display="off"/>
 <attribute name="NAME" x="10.652" y="67.2926" size="0.6096" layer="26" rot="MR270"/>
 <attribute name="VALUE" x="16.002" y="66.7766" size="0.6096" layer="28" rot="MR270"/>
 </element>
 <element name="LED1" library="led" library_urn="urn:adsk.eagle:library:259" package="SML0603" package3d_urn="urn:adsk.eagle:package:15832/1" value="" x="17.526" y="57.15" smashed="yes" rot="R90">
+<attribute name="DIGIKEY_NR" value="475-3118-1-ND " x="17.526" y="57.15" size="1.778" layer="27" rot="R90" display="off"/>
+<attribute name="DIGIKEY_PRICE" value="0.52 Fr." x="17.526" y="57.15" size="1.778" layer="27" rot="R90" display="off"/>
 <attribute name="NAME" x="16.526" y="56.15" size="1.27" layer="25" rot="R90"/>
 <attribute name="VALUE" x="19.526" y="56.15" size="1.27" layer="27" rot="R90"/>
@@
 </element>
 <element name="R2" library="rcl" library_urn="urn:adsk.eagle:library:334" package="R0603" package3d_urn="urn:adsk.eagle:package:23555/2" value="47" x="24.638" y="73.152" smashed="yes" rot="MR180">
+<attribute name="DIGIKEY_NR" value="311-470GRCT-ND" x="24.638" y="73.152" size="1.778" layer="28" rot="MR180" display="off"/>
+<attribute name="DIGIKEY_PRICE" value="0.1" x="24.638" y="73.152" size="1.778" layer="28" rot="MR180" display="off"/>
 <attribute name="NAME" x="24.003" y="72.517" size="1.27" layer="26" rot="MR180"/>
 <attribute name="SPICEPREFIX" value="R" x="70.358" y="118.872" size="1.778" layer="28" rot="MR180" display="off"/>
@@
 <element name="R9" library="rcl" library_urn="urn:adsk.eagle:library:334" package="R0603" package3d_urn="urn:adsk.eagle:package:23555/2" value="100" x="20.574" y="57.912" smashed="yes" rot="R180">
 <attribute name="DIGIKEY_NR" value="311-100DCT-ND" x="20.574" y="57.912" size="1.778" layer="27" rot="R180" display="off"/>
-<attribute name="DIGIKEY_PRIZE" value="0.20 Fr." x="20.574" y="57.912" size="1.778" layer="27" rot="R180" display="off"/>
+<attribute name="DIGIKEY_PRICE" value="0.20 Fr." x="20.574" y="57.912" size="1.778" layer="27" rot="R180" display="off"/>
 <attribute name="NAME" x="21.209" y="56.769" size="1.27" layer="25" rot="R180"/>
 <attribute name="SPICEPREFIX" value="R" x="-13.716" y="103.632" size="1.778" layer="27" rot="R180" display="off"/>
@@
 </element>
 <element name="R12" library="rcl" library_urn="urn:adsk.eagle:library:334" package="R0603" package3d_urn="urn:adsk.eagle:package:23555/2" value="4.7k" x="17.018" y="74.168" smashed="yes" rot="MR270">
+<attribute name="DIGIKEY_NR" value="311-4.70KHRCT-ND" x="17.018" y="74.168" size="1.778" layer="28" rot="MR270" display="off"/>
+<attribute name="DIGIKEY_PRICE" value="0.1" x="17.018" y="74.168" size="1.778" layer="28" rot="MR270" display="off"/>
 <attribute name="NAME" x="16.383" y="74.803" size="1.27" layer="26" rot="MR270"/>
 <attribute name="SPICEPREFIX" value="R" x="17.018" y="74.168" size="1.778" layer="28" rot="MR270" display="off"/>
@@
 <vertex x="-6.35" y="89.154"/>
 </polygon>
-<wire x1="11.766" y1="34.118" x2="17.526" y2="40.132" width="0.6096" layer="16"/>
-<wire x1="17.526" y1="40.132" x2="17.526" y2="51.308" width="0.6096" layer="16"/>
 <via x="17.526" y="51.308" extent="1-16" drill="0.35"/>
 <wire x1="17.526" y1="56.4" x2="17.526" y2="51.308" width="0.6096" layer="1"/>
@@
 <contactref element="X4" pad="1"/>
 <contactref element="R16" pad="1"/>
-<wire x1="10.0584" y1="50.21081875" x2="10.0584" y2="52.832" width="0.6096" layer="16"/>
 <wire x1="6.9596" y1="63.0564" x2="6.858" y2="63.158" width="0.6096" layer="16"/>
 <wire x1="8.128" y1="48.28041875" x2="8.128" y2="31.496" width="0.6096" layer="16"/>
 <wire x1="8.636" y1="30.988" x2="8.128" y2="31.496" width="0.6096" layer="16"/>
-<wire x1="8.128" y1="48.28041875" x2="10.0584" y2="50.21081875" width="0.6096" layer="16"/>
 <wire x1="6.9596" y1="60.07598125" x2="6.9596" y2="63.0564" width="0.6096" layer="16"/>
-<wire x1="10.0584" y1="52.832" x2="8.89" y2="54.0004" width="0.6096" layer="16"/>
 <wire x1="8.89" y1="54.0004" x2="8.89" y2="58.14558125" width="0.6096" layer="16"/>
 <wire x1="8.89" y1="58.14558125" x2="6.9596" y2="60.07598125" width="0.6096" layer="16"/>
+<wire x1="8.128" y1="48.28041875" x2="10.657790625" y2="50.810209375" width="0.6096" layer="16"/>
+<wire x1="10.657790625" y1="50.810209375" x2="10.657790625" y2="52.232609375" width="0.6096" layer="16"/>
+<wire x1="10.657790625" y1="52.232609375" x2="8.89" y2="54.0004" width="0.6096" layer="16"/>
 </signal>
 <signal name="N$18">
@@
 <wire x1="8.636" y1="28.21441875" x2="10.5664" y2="30.14481875" width="0.6096" layer="16"/>
 <wire x1="10.5664" y1="30.14481875" x2="10.5664" y2="31.83118125" width="0.6096" layer="16"/>
-<wire x1="14.8932" y1="54.19128125" x2="9.2456" y2="59.83888125" width="0.6096" layer="16"/>
+<wire x1="9.2456" y1="59.83888125" x2="11.555240625" y2="57.529240625" width="0.6096" layer="16"/>
 <wire x1="10.5664" y1="31.83118125" x2="9.65533125" y2="32.74225" width="0.6096" layer="16"/>
 <wire x1="9.2456" y1="59.83888125" x2="9.2456" y2="63.0564" width="0.6096" layer="16"/>
-<wire x1="14.8932" y1="46.39271875" x2="14.8932" y2="54.19128125" width="0.6096" layer="16"/>
-<wire x1="9.65533125" y1="32.74225" x2="9.65533125" y2="41.15485" width="0.6096" layer="16"/>
-<wire x1="9.65533125" y1="41.15485" x2="14.8932" y2="46.39271875" width="0.6096" layer="16"/>
+<wire x1="9.65533125" y1="41.15485" x2="9.65533125" y2="32.74225" width="0.6096" layer="16"/>
 <wire x1="9.2456" y1="63.0564" x2="9.227" y2="63.075" width="0.6096" layer="16"/>
+<wire x1="11.555240625" y1="57.529240625" x2="14.352759375" y2="57.529240625" width="0.6096" layer="16"/>
+<wire x1="14.352759375" y1="57.529240625" x2="14.732" y2="57.15" width="0.6096" layer="16"/>
+<wire x1="14.732" y1="57.15" x2="14.732" y2="46.23151875" width="0.6096" layer="16"/>
+<wire x1="14.732" y1="46.23151875" x2="9.65533125" y2="41.15485" width="0.6096" layer="16"/>
 </signal>
 <signal name="N$19">

Commit message: finished
Parts:
- added X6: MOLEX-8738-0343, ADC-Erweiterung:MOLEX-87438-0343
- moved R2 0.25 mm to (24.6, 73.4)
- moved R8 0.25 mm to (22.4, 19.8)
Connections:
- net N$10: now also X6.1, X6.1_1
- net N$8: now also X6.3, X6.3_1
- net N$9: now also X6.2, X6.2_1
Routing:
- net N$10: track 12.6 -> 33.5 mm
- net N$9: track 12.3 -> 27.1 mm
- net N$8: track 20.7 -> 33.1 mm
- net N$18: track 61.5 -> 60.5 mm
- net START: track 59.9 -> 60.6 mm
- net N$2: track 40.0 -> 40.5 mm

Commit message: Stand der Abgabe
Parts:
- moved R8 9.16 mm to (21.8, 29.0), flipped to the bottom
- moved X6 3.81 mm to (17.5, 84.3)
- moved R3 3.61 mm to (24.4, 21.3)
- moved C1 2.05 mm to (27.4, 83.3), flipped to the bottom
- moved R9 0.25 mm to (20.8, 57.9), flipped to the bottom, turned to 0 degrees
Routing:
- net DRDY: track 8.14 -> 19.8 mm
- net VCC: track 58.4 -> 49.1 mm, vias 0 -> 3
- net N$7: track 47.3 -> 38.3 mm, vias 1 -> 0
- net N$2: track 40.5 -> 44.7 mm
- net N$9: track 27.1 -> 30.9 mm
- net RESET: track 8.64 -> 5.30 mm
- net N$8: track 33.1 -> 36.0 mm
- net N$14: track 2.20 -> 4.99 mm, vias 0 -> 1
- net GND: track 10.7 -> 8.16 mm
- net N$10: track 33.5 -> 35.1 mm
- net MOSI: track 41.4 -> 41.7 mm, vias 0 -> 2
Other:
- board size 35.8 x 88.9 mm -> 35.5 x 88.9 mm
- board text added: "+3.3V"
- board text added: "1"
- board text added: "ADC-BOARD 2019 Noëmi Kurt Philipp Gurtner"
- board text added: "CS"
- board text added: "DRDY"
- board text added: "EX-IN_1"
- board text added: "EX-IN_2"
- board text added: "EX-IN_3"
- board text added: "GND"
- board text added: "MISO"
- board text added: "MOSI"
- board text added: "PT100"
- board text added: "RESET"
- board text added: "SCLK"
- board text added: "START"
