File: ADC-Erweiterung/V0.2.brd (EAGLE design)
At the start: 35.5 x 88.9 mm, 28 parts, among them IC1 ADS124S06IPBS, X1 33PIN-2.54, X2 MKDSN1,5/3-5,08, X3 A97581-ND, X4 A97581-ND, X5 A97581-ND, X6 MOLEX-8738-0343

Commit message: Software Start & Aufgeräumt
Connections:
- net GND: now also IC1.1
Changed lines of the file:
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@@
 <wire x1="27.432" y1="82.462" x2="30.441" y2="82.462" width="0.6096" layer="16"/>
 <wire x1="30.441" y1="82.462" x2="30.48" y2="82.423" width="0.6096" layer="16"/>
+<contactref element="IC1" pad="1"/>
 </signal>
 <signal name="N$1">
