File: ADC-Erweiterung/V0.2.sch (EAGLE design)
At the start: 28 parts, among them IC1 ADS124S06IPBS, X1 33PIN-2.54, X2 MKDSN1,5/3-5,08, X3 A97581-ND, X4 A97581-ND, X5 A97581-ND, X6 MOLEX-8738-0343

Commit message: Software Start & Aufgeräumt
Connections:
- net GND: now also IC1.AINCOM
Other:
- note added: "3V GND VBAT PC13 PC14 PC15 PF0 PF1 GND NRST PC0 PC1 PC2 PC3 PA0 PA1 PA2 PA3 PF4 PF5 PA4 PA5 PA6 PA7 PC4 PC5 PB0 PB1 PB2 PB10 PB11 PB12 GND"
- note removed: "3V GND VBAT PC13 PC14 PC15 PF0 PF1 GND NRST PC0 PC1 PC2 PC3 PA0 PA1 PA2 PA3 PF4 PF5 PA4 PA5 PA6 PA7 PC4 PC5 PB0 PB1 PB2 PB10 PB11 PB1 GND"
Changed lines of the file:
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@@
 <sheet>
 <plain>
-<text x="184.15" y="17.78" size="1.6383" layer="91">3V
+<text x="186.69" y="17.78" size="1.6383" layer="91">3V
 GND
 VBAT
@@
 PB10
 PB11
-PB1
+PB12
 GND</text>
 <wire x1="-3.81" y1="92.71" x2="-3.81" y2="77.47" width="0.1524" layer="90"/>
@@
 <wire x1="102.87" y1="41.91" x2="107.95" y2="41.91" width="0.1524" layer="91"/>
 <junction x="107.95" y="41.91"/>
-</segment>
-<segment>
+<pinref part="IC1" gate="G$1" pin="AINCOM"/>
+<wire x1="97.79" y1="44.196" x2="97.79" y2="41.91" width="0.1524" layer="91"/>
+<wire x1="97.79" y1="41.91" x2="102.87" y2="41.91" width="0.1524" layer="91"/>
+<junction x="102.87" y="41.91"/>
+</segment>
+<segment>
