File: ADC-Erweiterung/V02/V0.2.brd (EAGLE design)
At the start: 35.5 x 88.9 mm, 28 parts, among them IC1 ADS124S06IPBS, X1 33PIN-2.54, X2 MKDSN1,5/3-5,08, X3 A97581-ND, X4 A97581-ND, X5 A97581-ND, X6 MOLEX-8738-0343

Commit message: SchemativV02
Parts:
- removed LED1: (no value), led:SML0603
- removed R10, R12, R13, R14, R15, R16, R17: 4.7k, rcl:R0603
- removed R11: 2k2, rcl:R0805W
- removed R3, R6, R8: 47, rcl:R0603
- removed X2: MKDSN1,5/3-5,08, ADC-Erweiterung:MKDSN1,5/3-5,08
- removed X6: MOLEX-8738-0343, ADC-Erweiterung:MOLEX-87438-0343
- added C101, C102, C104, C105: 1u, rcl:C0603
- added LED101: (no value), led:SML0603
- added R101, R104, R106, R108: 2k2, rcl:R0805W
- added R102: 4.7k, rcl:R0603
- added R103, R105, R107: 47k, rcl:R0603
- added R110, R113, R115: 47, rcl:R0603
- added SV101: (no value), con-lstb:MA08-1
- added X101: MOLEX-8738-0343, ADC-Erweiterung:MOLEX-87438-0343
- renumbered C1 to C103, C2 to C106, C3 to C108, C4 to C107, IC1 to IC101, R2 to R109, R4 to R111, R5 to R112, R7 to R114, R9 to R116, X1 to X105, X3 to X104, X4 to X103, X5 to X102
Connections:
- removed net N$10: R11.2, R14.1, X2.3, X6.1, X6.1_1
- removed net N$12: IC101.3, R16.2
- removed net N$13: IC101.2, R17.2
- removed net N$16: IC101.4, R15.2
- removed net N$19: IC101.5, R14.2
- removed net N$20: IC101.7, R12.2
- removed net N$21: IC101.6, R13.2
- removed net N$8: R10.1, R12.1, X2.1, X6.3, X6.3_1
- removed net N$9: R13.1, X2.2, X6.2, X6.2_1
- new net AIN0: C104.1, C105.1, IC101.7, R102.1, X101.3, X101.3_1
- new net AIN1: C102.1, C104.2, IC101.6, X101.2, X101.2_1
- new net AIN2: C101.1, IC101.5, R101.2, X101.1, X101.1_1
- net CS: now also SV101.1
- net DRDY: now also R115.2, SV101.7; no longer R8.2
- net GND: now also C101.2, C102.2, C105.2, LED101.C, R101.1, R104.1, R106.1, R108.1, SV101.8; no longer LED1.C, R11.1
- net MISO: now also R113.2, SV101.3; no longer R6.2
- net MOSI: now also SV101.4
- net N$11: now also IC101.4, R103.1, R104.2; no longer R15.1
- net N$14: now also LED101.A; no longer LED1.A
- net N$17: now also IC101.3, R105.1, R106.2; no longer R16.1
- net N$18: now also IC101.2, R107.1, R108.2; no longer R17.1
- net N$2: now also R110.1; no longer R3.1
- net N$5: now also R113.1; no longer R6.1
- net N$7: now also R115.1; no longer R8.1
- net RESET: now also R110.2, SV101.6; no longer R3.2
- net SCLK: now also SV101.2
- net START: now also SV101.5
- net VCC: now also R102.2, R103.2, R105.2, R107.2; no longer R10.2
Routing:
- net VCC: track 49.1 -> 109.2 mm, vias 3 -> 2
- net N$8: track 36.0 -> 0.00 mm
- net N$10: track 35.1 -> 0.00 mm
- net AIN0: track 0.00 -> 32.3 mm, vias 0 -> 1
- net N$9: track 30.9 -> 0.00 mm
- net N$11: track 13.3 -> 42.6 mm
- net AIN1: track 0.00 -> 28.3 mm, vias 0 -> 1
- net N$17: track 35.0 -> 61.9 mm
- net RESET: track 5.30 -> 31.4 mm
- net N$18: track 60.5 -> 85.1 mm
- net N$2: track 44.7 -> 21.3 mm
- net AIN2: track 0.00 -> 22.8 mm, vias 0 -> 1
- net DRDY: track 19.8 -> 39.3 mm
- net MOSI: track 39.9 -> 58.4 mm
- net GND: track 8.16 -> 26.6 mm, vias 1 -> 13
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- added copper zone on layer 1, net GND
Other:
- board text added: "ADC-BOARD 2019 V2.0 Noëmi Kurt Philipp Gurtner"
- board text removed: "ADC-BOARD 2019 Noëmi Kurt Philipp Gurtner"

Commit message: AbgabeSoftware
Connections:
- new net N$8: R104.1
- new net N$9: R106.1
- net GND: no longer R104.1, R106.1
Routing:
- net GND: track 26.6 -> 12.2 mm, vias 13 -> 83
- net AIN2: track 22.8 -> 24.3 mm
- net AIN1: track 28.3 -> 29.7 mm
- net START: track 71.6 -> 70.8 mm
Other:
- board text added: "+3V"
- board text added: "ADC-BOARD 2019 V0.2 Noëmi Kurt Philipp Gurtner"
- board text removed: "+3.3V"
- board text removed: "ADC-BOARD 2019 V2.0 Noëmi Kurt Philipp Gurtner"

Commit message: improuveschematic
Connections:
- removed net N$8: R104.1
- removed net N$9: R106.1
- net GND: now also R104.1, R106.1
Changed lines of the file:
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@@
 <setting verticaltext="up"/>
 </settings>
-<grid distance="10" unitdist="mil" unit="mm" style="dots" multiple="1" display="yes" altdistance="5" altunitdist="mil" altunit="mil"/>
+<grid distance="50" unitdist="mil" unit="mil" style="dots" multiple="1" display="yes" altdistance="5" altunitdist="mil" altunit="mil"/>
 <layers>
-<layer number="1" name="Top" color="4" fill="1" visible="no" active="yes"/>
+<layer number="1" name="Top" color="4" fill="1" visible="yes" active="yes"/>
 <layer number="2" name="Route2" color="16" fill="1" visible="no" active="no"/>
 <layer number="3" name="Route3" color="17" fill="1" visible="no" active="no"/>
@@
 <layer number="14" name="Route14" color="22" fill="1" visible="no" active="no"/>
 <layer number="15" name="Route15" color="23" fill="1" visible="no" active="no"/>
-<layer number="16" name="Bottom" color="1" fill="1" visible="yes" active="yes"/>
+<layer number="16" name="Bottom" color="1" fill="1" visible="no" active="yes"/>
 <layer number="17" name="Pads" color="2" fill="1" visible="yes" active="yes"/>
-<layer number="18" name="Vias" color="2" fill="1" visible="yes" active="yes"/>
+<layer number="18" name="Vias" color="2" fill="1" visible="no" active="yes"/>
 <layer number="19" name="Unrouted" color="6" fill="1" visible="yes" active="yes"/>
 <layer number="20" name="Dimension" color="24" fill="1" visible="yes" active="yes"/>
-<layer number="21" name="tPlace" color="7" fill="1" visible="no" active="yes"/>
-<layer number="22" name="bPlace" color="7" fill="1" visible="yes" active="yes"/>
+<layer number="21" name="tPlace" color="7" fill="1" visible="yes" active="yes"/>
+<layer number="22" name="bPlace" color="7" fill="1" visible="no" active="yes"/>
 <layer number="23" name="tOrigins" color="15" fill="1" visible="no" active="yes"/>
-<layer number="24" name="bOrigins" color="15" fill="1" visible="yes" active="yes"/>
-<layer number="25" name="tNames" color="7" fill="1" visible="no" active="yes"/>
-<layer number="26" name="bNames" color="7" fill="1" visible="yes" active="yes"/>
+<layer number="24" name="bOrigins" color="15" fill="1" visible="no" active="yes"/>
+<layer number="25" name="tNames" color="7" fill="1" visible="yes" active="yes"/>
+<layer number="26" name="bNames" color="7" fill="1" visible="no" active="yes"/>
 <layer number="27" name="tValues" color="7" fill="1" visible="no" active="yes"/>
 <layer number="28" name="bValues" color="7" fill="1" visible="no" active="yes"/>
@@
 <layer number="38" name="bTest" color="7" fill="1" visible="no" active="yes"/>
 <layer number="39" name="tKeepout" color="4" fill="11" visible="no" active="yes"/>
-<layer number="40" name="bKeepout" color="1" fill="11" visible="yes" active="yes"/>
+<layer number="40" name="bKeepout" color="1" fill="11" visible="no" active="yes"/>
 <layer number="41" name="tRestrict" color="4" fill="10" visible="no" active="yes"/>
-<layer number="42" name="bRestrict" color="1" fill="10" visible="yes" active="yes"/>
+<layer number="42" name="bRestrict" color="1" fill="10" visible="no" active="yes"/>
 <layer number="43" name="vRestrict" color="2" fill="10" visible="no" active="yes"/>
 <layer number="44" name="Drills" color="7" fill="1" visible="no" active="yes"/>
@@
 <layer number="48" name="Document" color="7" fill="1" visible="no" active="yes"/>
 <layer number="49" name="Reference" color="7" fill="1" visible="no" active="yes"/>
-<layer number="51" name="tDocu" color="7" fill="1" visible="no" active="yes"/>
-<layer number="52" name="bDocu" color="7" fill="1" visible="yes" active="yes"/>
+<layer number="51" name="tDocu" color="7" fill="1" visible="yes" active="yes"/>
+<layer number="52" name="bDocu" color="7" fill="1" visible="no" active="yes"/>
 <layer number="88" name="SimResults" color="9" fill="1" visible="no" active="no"/>
 <layer number="89" name="SimProbes" color="9" fill="1" visible="no" active="no"/>
@@
 <text x="28.194" y="83.312" size="1.5" layer="25" rot="R180">GND</text>
 <text x="21.336" y="17.78" size="1.5" layer="25">DRDY</text>
-<text x="21.336" y="20.32" size="1.5" layer="25">RESET</text>
-<text x="24.638" y="19.812" size="1.5" layer="25">START</text>
+<text x="21.59" y="20.447" size="1.5" layer="25">RESET</text>
+<text x="21.463" y="22.987" size="1.5" layer="25">START</text>
 <text x="21.336" y="33.02" size="1.5" layer="25">CS</text>
-<text x="24.638" y="24.892" size="1.5" layer="25">MISO</text>
-<text x="24.638" y="27.432" size="1.5" layer="25">SCLK</text>
-<text x="24.638" y="22.352" size="1.5" layer="25">MOSI</text>
+<text x="21.463" y="27.94" size="1.5" layer="25">MISO</text>
+<text x="21.336" y="30.607" size="1.5" layer="25">SCLK</text>
+<text x="21.59" y="25.4" size="1.5" layer="25">MOSI</text>
 <text x="5.334" y="59.69" size="1.5" layer="25">EX-IN_1</text>
 <text x="5.08" y="38.862" size="1.5" layer="25">EX-IN_2</text>
@@
 <wire x1="19.558" y1="21.082" x2="17.78" y2="21.082" width="0.6096" layer="16"/>
 <wire x1="17.78" y1="21.082" x2="16.256" y2="22.606" width="0.6096" layer="16"/>
-<wire x1="30.48" y1="21.463" x2="30.099" y2="21.082" width="0.6096" layer="16"/>
-<wire x1="30.099" y1="21.082" x2="19.558" y2="21.082" width="0.6096" layer="16"/>
+<wire x1="19.558" y1="21.082" x2="19.939" y2="21.463" width="0.6096" layer="1"/>
+<wire x1="19.939" y1="21.463" x2="30.48" y2="21.463" width="0.6096" layer="1"/>
 </signal>
 <signal name="DRDY">
@@
 <contactref element="C102" pad="2"/>
 <contactref element="C105" pad="2"/>
-<contactref element="R108" pad="1"/>
 <contactref element="SV101" pad="8"/>
-<wire x1="5.2975" y1="19.812" x2="5.506" y2="19.6035" width="0.6096" layer="1"/>
 <wire x1="5.506" y1="19.6035" x2="5.506" y2="12.02" width="0.6096" layer="1"/>
 <polygon width="0.6096" layer="1" spacing="0.254">
@@
 <via x="32.258" y="20.574" extent="1-16" drill="0.35"/>
 <via x="25.4" y="12.192" extent="1-16" drill="0.35"/>
+<contactref element="R104" pad="1"/>
+<contactref element="R106" pad="1"/>
+<contactref element="R108" pad="1"/>
 </signal>
 <signal name="N$1">
@@
 <signal name="N$15">
 <contactref element="IC101" pad="23"/>
+<wire x1="13.482" y1="60.452" x2="13.482" y2="59.758" width="0.3048" layer="16"/>
+<wire x1="13.482" y1="61.924" x2="13.482" y2="60.452" width="0.254" layer="16"/>
 <contactref element="C108" pad="1"/>
-<wire x1="13.482" y1="60.452" x2="13.482" y2="59.758" width="0.3048" layer="16"/>
-<wire x1="13.482" y1="59.758" x2="13.804" y2="59.436" width="0.3048" layer="16"/>
-<wire x1="13.482" y1="61.924" x2="13.482" y2="60.452" width="0.254" layer="16"/>
+<wire x1="13.804" y1="59.436" x2="13.482" y2="59.758" width="0" layer="19" extent="16-16"/>
 </signal>
 <signal name="N$17">
@@
 <wire x1="15.4336" y1="70.9886125" x2="15.4336" y2="68.1964" width="0.2032" layer="16"/>
 </signal>
-<signal name="N$8" class="1">
-<contactref element="R104" pad="1"/>
-</signal>
-<signal name="N$9" class="1">
-<contactref element="R106" pad="1"/>
-</signal>
 </signals>
