File: ADC-Erweiterung/V02/V0.2.sch (EAGLE design)
At the start: 28 parts, among them IC1 ADS124S06IPBS, X1 33PIN-2.54, X2 MKDSN1,5/3-5,08, X3 A97581-ND, X4 A97581-ND, X5 A97581-ND, X6 MOLEX-8738-0343

Commit message: SchemativV02
Parts:
- removed R11: 2k2, rcl:R-EU_R0805W
- removed R12, R13, R14, R15, R16, R17: 4.7k, rcl:R-EU_R0603
- removed X2: MKDSN1,5/3-5,08, ADC-Erweiterung:MKDSN1,5/3-5,08
- removed X3, X4, X5: A97581-ND, ADC-Erweiterung:A97581-ND
- removed X6: MOLEX-8738-0343, ADC-Erweiterung:MOLEX-8738-0343
- added C101, C102, C104, C105: 1u, rcl:C-EUC0603
- added R101, R104, R106, R108: 2k2, rcl:R-EU_R0805W
- added R103, R105, R107: 47k, rcl:R-EU_R0603
- added SV101: (no value), con-lstb:MA08-1
- added X101: MOLEX-8738-0343, ADC-Erweiterung:MOLEX-8738-0343
- added X102, X103, X104: A97581-ND, ADC-Erweiterung:A97581-ND
- renumbered C1 to C103, C2 to C106, C3 to C108, C4 to C107, IC1 to IC101, LED1 to LED101, R10 to R102, R2 to R109, R3 to R110, R4 to R111, R5 to R112, R6 to R113, R7 to R114, R8 to R115, R9 to R116, X1 to X105
Connections:
- removed net N$10: R11.2, R14.1, X2-3.KL, X6.1
- removed net N$12: IC101.AIN4, R16.2
- removed net N$13: IC101.AIN5, R17.2
- removed net N$16: IC101.AIN3, R15.2
- removed net N$19: IC101.AIN2, R14.2
- removed net N$20: IC101.AIN0, R12.2
- removed net N$21: IC101.AIN1, R13.2
- removed net N$8: R102.1, R12.1, X2-1.KL, X6.3
- removed net N$9: R13.1, X2-2.KL, X6.2
- new net AIN0: C104.1, C105.1, IC101.AIN0, R102.1, X101.3
- new net AIN1: C102.1, C104.2, IC101.AIN1, X101.2
- new net AIN2: C101.1, IC101.AIN2, R101.2, X101.1
- net CS: now also SV101.1
- net DRDY: now also SV101.7
- net GND: now also C101.2, C102.2, C105.2, R101.1, R104.1, R106.1, R108.1, SV101.8, X102.2, X103.2, X104.2; no longer R11.1, X3.2, X4.2, X5.2
- net MISO: now also SV101.3
- net MOSI: now also SV101.4
- net N$11: now also IC101.AIN3, R103.1, R104.2, X102.1; no longer R15.1, X5.1
- net N$17: now also IC101.AIN4, R105.1, R106.2, X103.1; no longer R16.1, X4.1
- net N$18: now also IC101.AIN5, R107.1, R108.2, X104.1; no longer R17.1, X3.1
- net RESET: now also SV101.6
- net SCLK: now also SV101.2
- net START: now also SV101.5
- net VCC: now also R103.2, R105.2, R107.2
Other:
- note removed: "PT100"

Commit message: AbgabeSoftware
Parts:
- SV101: DIGIKEY_NR (none) -> 732-5321-ND; DIGIKEY_PRICE (none) -> 0.37
Connections:
- new net N$8: R104.1
- new net N$9: R106.1
- net GND: no longer R104.1, R106.1
Other:
- moved on the sheet: C101, C102, R101, R102, R103, R104, R105, R106, R107, R108, X101, X102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

Commit message: improuveschematic
Connections:
- removed net N$8: R104.1
- removed net N$9: R106.1
- net GND: now also R104.1, R106.1
Other:
- moved on the sheet: C101, C102, C103, C104, C105, C106, C107, C108, IC101, LED101, R101, R102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
