File: Hardware/V02/V0.2.brd (EAGLE design)
At the start: 35.5 x 88.9 mm, 32 parts, among them IC101 ADS124S06IPBS, X101 MOLEX-8738-0343, X102 A97581-ND, X103 A97581-ND, X104 A97581-ND, X105 33PIN-2.54

Commit message: Schemaänderung; BNC-Abschwächer
Parts:
- moved R104 20.2 mm to (3.68, 63.4)
- moved R103 16.4 mm to (5.80, 63.8), turned to 270 degrees
- moved R106 3.94 mm to (10.0, 42.5)
- moved R105 0.75 mm to (10.5, 40.4), turned to 180 degrees
- moved R107 0.13 mm to (10.0, 19.8), turned to 180 degrees
Connections:
- new net N$12: R103.2, X102.1
- new net N$13: R105.2, X103.1
- new net N$16: R107.2, X104.1
- net N$11: no longer X102.1
- net N$17: no longer X103.1
- net N$18: no longer X104.1
- net VCC: no longer R103.2, R105.2, R107.2
Routing:
- net VCC: track 109.2 -> 50.4 mm
- net N$11: track 42.6 -> 19.2 mm, vias 0 -> 1
- net N$18: track 85.1 -> 65.6 mm, vias 0 -> 1
- net N$17: track 61.9 -> 44.1 mm, vias 0 -> 1
- net N$12: track 0.00 -> 12.6 mm
- net N$16: track 0.00 -> 11.1 mm
- net N$13: track 0.00 -> 9.84 mm
- net GND: track 11.9 -> 14.6 mm, vias 83 -> 82
